Commit message: Added pot to the scenario and adjusted it's handle positions and it's mass
The pot was far too heavy (~10kg) and the handles were too close to it's center. Readded the pot to do experiments with two-handled objects and adjusted the mass and handles accordingly.

File: models/Cookingpot_2.urdf (robot description, URDF)
Before this commit: robot Cookingpot_2, 1 links, 0 joints
Links:
- link body: mass 10 -> 0.5
