Commit message: Moved table URDF to origin and fixed coordinates in launch file.

File: models/table.urdf (robot description, URDF)
Before this commit: robot table, 5 links, 4 joints
Joints:
- joint leg1_joint: origin xyz=1.48 1.0 0.55 rpy=0 0 0 -> xyz=0.5 1.0 0.55 rpy=0 0 0
- joint leg2_joint: origin xyz=0.48 1.0 0.55 rpy=0 0 0 -> xyz=-0.5 1.0 0.55 rpy=0 0 0
- joint leg3_joint: origin xyz=1.48 -1.0 0.55 rpy=0 0 0 -> xyz=0.5 -1.0 0.55 rpy=0 0 0
- joint leg4_joint: origin xyz=0.48 -1.0 0.55 rpy=0 0 0 -> xyz=-0.5 -1.0 0.55 rpy=0 0 0
